File: hardware/noise/noise.kicad_sch (KiCad schematic)
At the start: 66 parts, among them J1 Conn_02x05_Odd_Even, J2 White, J3 Pink, J4 Blue, J5 Grainy, J6 HP Grainy, Q1 BC547, U1 TL074, U2 TL072

Commit message: Doc cleanup, assembly guide, faceplate art
Parts:
- C9, J6, R32: now fitted
Changed lines of the file:
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@@
 		(in_bom yes)
 		(on_board yes)
-		(dnp yes)
+		(dnp no)
 		(fields_autoplaced yes)
 		(property "Reference" "J6"
@@
 		(in_bom yes)
 		(on_board yes)
-		(dnp yes)
+		(dnp no)
 		(property "Reference" "R32"
 			(at 154.94 167.6399 0)
@@
 		(in_bom yes)
 		(on_board yes)
-		(dnp yes)
+		(dnp no)
 		(fields_autoplaced yes)
 		(property "Reference" "C9"
